File: oscillogoat_0.1.kicad_pcb (KiCad board)
At the start: 2 copper layers, 308 parts, among them IC1 XC7A12T-1CPG238C, IC2 FT602Q-B-T, IC5 ADC09DJ800AAV, J1002_1 BNC, J3_1 UFL, J4_1 UFL, Q1 DMN62D0UW, Q2 DMN62D0UW, U1001_1 TMUX4053, U1008_1 LMH6518, U1009_1 BUF802, U1011_1 OPA140AIDBVR, U13 LM27761, U14 TPS7A9101, U15 TPS7A9101, U16 TPS7A2033, U17 TPS61023, U18 TPS7A9101, U19 MX25L6433FZNI-08G, U2 MCP4452-104E, U20 TPS62A02, U21 TPS62A02, U22 TPS7A9101, U23 TPS62A02, U24 TPS62A02, U3 MCP4728, U4 REF2025, U5 OPA140AIDBVR, U8 TPS62A02, Y1 ASEMPLV-100.000MHZ-LR-T

Commit message: update
Parts:
- removed C1001_1, C186: 100pF, Thunderscope_Rev5:GEN_C_0402
- removed C103, C1036_1, C1037_1, C61, C65, C79: 1uF, Thunderscope_Rev5:GEN_C_0402
- removed C1031_1: 10nF, Thunderscope_Rev5:GEN_C_0603
- removed C1039_1, C153, C187: 10uF, Thunderscope_Rev5:GEN_C_0603
- removed C188, C97, C98: 22uF, Thunderscope_Rev5:GEN_C_0805
- removed FB1000_1, R91: 120@100MHZ, Thunderscope_Rev5:GEN_R_0402
- removed J3_1, J4_1: UFL, Thunderscope_Rev5:TE_2334884-1
- removed L4: 1uH, Thunderscope_Rev5:GEN_L_1210
- removed R101, R108, R114, R115, R133, R135: 0R1, Thunderscope_Rev5:GEN_R_0402
- removed R1052_1, R128, R129, R130: 10K, Thunderscope_Rev5:GEN_R_0402
- removed R126: 0.01, Thunderscope_Rev5:GEN_R_0603
- removed R70: 4.7K, Thunderscope_Rev5:GEN_R_0402
- removed TP1016_1, TP1018_1, TP29, TP31, TP35, TP39, TP4, TP67, TP68: PCB, Thunderscope_Rev5:GEN_TP_PCB
- removed U1001_1: TMUX4053, Thunderscope_Rev5:TI_TSOT-23-16_DYY0016A
- removed U23: TPS62A02, Thunderscope_Rev5:TI_SOT563_DRL0006A
- added C1: 100u, Passives_SMD:1206_3216Metric, F.Cu at (180.4, 74.6)
- added C1007_2: 10uF, Passives_SMD:0603_1608Metric, F.Cu at (161.5, 141.4)
- added C1007_3: 10uF, Passives_SMD:0603_1608Metric, F.Cu at (153.9, 141.3)
- added C1008_2: 10uF, Passives_SMD:0603_1608Metric, F.Cu at (163.8, 145.5)
- added C13: 100u, Passives_SMD:1206_3216Metric, F.Cu at (167.7, 68.5)
- added C138: 1uF, Passives_SMD:0402_1005Metric, B.Cu at (59.4, 58.0)
- added C139: 1uF, Passives_SMD:0402_1005Metric, B.Cu at (59.8, 58.9)
- added C14: 100u, Passives_SMD:1206_3216Metric, F.Cu at (153.8, 45.6)
- added C140: 1uF, Passives_SMD:0402_1005Metric, B.Cu at (60.1, 59.9)
- added C142: 10uF, Passives_SMD:0603_1608Metric, F.Cu at (38.4, 51.1)
- added C143: 10uF, Passives_SMD:0603_1608Metric, F.Cu at (44.1, 44.6)
- added C15: 100u, Passives_SMD:1206_3216Metric, F.Cu at (162.0, 45.7)
- added C154: 47uF, Passives_SMD:0805_2012Metric, F.Cu at (40.5, 67.2)
- added C155: 47uF, Passives_SMD:0805_2012Metric, F.Cu at (36.8, 41.1)
- added C16: 100u, Passives_SMD:1206_3216Metric, F.Cu at (162.4, 54.2)
- added C163: 1uF, Passives_SMD:0402_1005Metric, B.Cu at (55.4, 58.1)
- added C164: 1uF, Passives_SMD:0402_1005Metric, B.Cu at (57.3, 59.6)
- added C165: 1uF, Passives_SMD:0402_1005Metric, B.Cu at (46.8, 68.1)
- added C166: 10uF, Passives_SMD:0603_1608Metric, F.Cu at (42.5, 51.1)
- added C167: 10uF, Passives_SMD:0603_1608Metric, F.Cu at (48.3, 44.6)
- added C168: 47uF, Passives_SMD:0805_2012Metric, F.Cu at (36.8, 44.1)
- added C169: 10uF, Passives_SMD:0603_1608Metric, F.Cu at (48.3, 47.2)
- added C17: 100u, Passives_SMD:1206_3216Metric, F.Cu at (29.1, 55.1)
- added C170: 10uF, Passives_SMD:0603_1608Metric, F.Cu at (48.3, 49.8)
- added C171: 1uF, Passives_SMD:0402_1005Metric, B.Cu at (49.0, 67.4)
- added C172: 1uF, Passives_SMD:0402_1005Metric, B.Cu at (59.9, 57.0)
- added C173: 1uF, Passives_SMD:0402_1005Metric, B.Cu at (55.1, 55.6)
- added C18: 100u, Passives_SMD:1206_3216Metric, F.Cu at (29.1, 58.4)
- added C19: 100u, Passives_SMD:1206_3216Metric, F.Cu at (168.6, 139.9)
- added C192: 1uF, Passives_SMD:0402_1005Metric, B.Cu at (59.2, 55.8)
- added C194: 1uF, Passives_SMD:0402_1005Metric, B.Cu at (59.7, 54.8)
- added C195: 47uF, Passives_SMD:0805_2012Metric, F.Cu at (41.5, 47.2)
- added C196: 1uF, Passives_SMD:0402_1005Metric, B.Cu at (56.2, 60.6)
- added C20: 100u, Passives_SMD:1206_3216Metric, F.Cu at (160.7, 139.5)
- added C21: 100u, Passives_SMD:1206_3216Metric, F.Cu at (153.1, 139.4)
- added C81: 1uF, Passives_SMD:0402_1005Metric, B.Cu at (57.1, 55.5)
- added C83: 1uF, Passives_SMD:0402_1005Metric, B.Cu at (48.3, 54.2)
- added C84: 1uF, Passives_SMD:0402_1005Metric, B.Cu at (48.7, 57.1)
- added C86: 1uF, Passives_SMD:0402_1005Metric, B.Cu at (48.8, 60.6)
- added F1: 120@100MHZ, Passives_SMD:0402_1005Metric, F.Cu at (179.3, 76.6)
- added F10: 120@100MHZ, Passives_SMD:0402_1005Metric, F.Cu at (159.1, 141.1)
- added F11: 120@100MHZ, Passives_SMD:0402_1005Metric, F.Cu at (151.5, 141.0)
- added F2: 120@100MHZ, Passives_SMD:0402_1005Metric, F.Cu at (177.3, 76.6)
- added F3: 120@100MHZ, Passives_SMD:0402_1005Metric, F.Cu at (167.2, 70.4)
- added F4: 120@100MHZ, Passives_SMD:0402_1005Metric, F.Cu at (153.9, 47.5)
- added F5: 120@100MHZ, Passives_SMD:0402_1005Metric, F.Cu at (161.6, 47.6)
- added F6: 120@100MHZ, Passives_SMD:0402_1005Metric, F.Cu at (162.0, 56.1)
- added F7: 120@100MHZ, Passives_SMD:0402_1005Metric, F.Cu at (29.6, 45.0)
- added F8: 120@100MHZ, Passives_SMD:0402_1005Metric, F.Cu at (29.6, 47.1)
- added F9: 120@100MHZ, Passives_SMD:0402_1005Metric, F.Cu at (167.0, 141.5)
- added J5: 2.54mm 6 Pin TH, Thunderscope_Rev5:GEN_2.54MM_6_PIN_TH_RA, F.Cu at (91.4, 25.3)
- added R136: 4.7K, Passives_SMD:0402_1005Metric, F.Cu at (87.3, 31.8)
- added R137: 4.7K, Passives_SMD:0402_1005Metric, F.Cu at (87.3, 33.8)
- added R138: 4.7K, Passives_SMD:0402_1005Metric, F.Cu at (87.3, 35.9)
- added R139: 4.7K, Passives_SMD:0402_1005Metric, F.Cu at (87.3, 38.0)
- added R140: 4.7K, Passives_SMD:0402_1005Metric, F.Cu at (87.3, 40.1)
- added R141: 0R1, Passives_SMD:0402_1005Metric, F.Cu at (34.6, 50.5)
- added R143: 100, Passives_SMD:0402_1005Metric, F.Cu at (88.4, 47.0)
- added R3: DNP, Passives_SMD:0402_1005Metric, F.Cu at (75.4, 27.6)
- added R4: DNP (place for LED), Passives_SMD:0402_1005Metric, F.Cu at (75.4, 29.7)
- added S1: 416131160803, Snapeda:416131160803, F.Cu at (76.7, 38.1)
- added TP75: PCB, Thunderscope_Rev5:GEN_TP_PCB, F.Cu at (108.2, 33.8)
- added TP76: PCB, Thunderscope_Rev5:GEN_TP_PCB, F.Cu at (108.2, 36.3)
- added TP77: PCB, Thunderscope_Rev5:GEN_TP_PCB, F.Cu at (108.2, 38.7)
- added TP78: PCB, Thunderscope_Rev5:GEN_TP_PCB, F.Cu at (110.6, 21.6)
- C10: value 10uF -> 100u; footprint Thunderscope_Rev5:GEN_C_0603 -> Passives_SMD:1206_3216Metric
- C100, C1002_1, C102, C1032_1, C1033_1, C1034_1, C1035_1, C1038_1, C1041_1, C1042_1, C1043_1, C1044_1, C1045_1, C1046_1, C1047_1, C1048_1, C1049_1, C1050_1, C1052_1, C1053_1, C1054_1, C1055_1, C1056_1, C1057_1, C11, C112, C123, C124, C125, C126, C127, C129, C132, C174, C178, C185, C190, C2, C3, C4, C5, C6, C7, C74, C76, C8, C82: footprint Thunderscope_Rev5:GEN_C_0402 -> Passives_SMD:0402_1005Metric
- C1003_1, C1004_1, C1005_1, C1006_1, C1007_1, C1008_1, C1030_1, C1040_1, C106, C111, C114, C115, C116, C117, C119, C12, C120, C121, C122, C130, C131, C133, C144, C145, C146, C148, C149, C150, C151, C152, C175, C179, C181, C182, C183, C184, C189, C71, C72, C73, C85, C9, C93, C94, C95, C96: footprint Thunderscope_Rev5:GEN_C_0603 -> Passives_SMD:0603_1608Metric
- C101, C104, C105, C128, C176, C177, C180, C191, C75, C99: footprint Thunderscope_Rev5:GEN_C_0805 -> Passives_SMD:0805_2012Metric
- C147: value 10uF -> 1uF; footprint Thunderscope_Rev5:GEN_C_0603 -> Passives_SMD:0402_1005Metric; moved to B.Cu
- C55, C56, C57, C58, C59, C60, C62, C63, C64, C66, C67, C68, C69, C70, C77, C78, C80: footprint Thunderscope_Rev5:GEN_C_0402 -> Passives_SMD:0402_1005Metric; moved to B.Cu
- FB1001_1, R1, R10, R100, R102, R1033_1, R1036_1, R1037_1, R1039_1, R104, R1041_1, R1042_1, R1043_1, R1044_1, R1045_1, R1046_1, R1047_1, R1048_1, R105, R106, R107, R109, R11, R110, R111, R112, R113, R117, R118, R119, R12, R121, R122, R124, R125, R127, R131, R132, R52_1, R55, R56, R66, R67, R68, R69, R71, R72, R9, R90, R93, R96, R97_1, R99: footprint Thunderscope_Rev5:GEN_R_0402 -> Passives_SMD:0402_1005Metric
- L1, L2, L3, L5, L6: footprint Thunderscope_Rev5:GEN_L_1210 -> Passives_SMD:1210_3225Metric
- R1003_1, R1022_1, R1035_1, R1038_1: footprint Thunderscope_Rev5:GEN_R_0603 -> Passives_SMD:0603_1608Metric
- R103, R116, R120, R123, R134, R14, R57, R97, R98: value 0.01 -> 0R01; footprint Thunderscope_Rev5:GEN_R_0603 -> Passives_SMD:0603_1608Metric
- moved U14 214.9 mm to (244.5, 66.5)
- moved C123 201.7 mm to (246.8, 67.1), turned to 90 degrees
- moved C115 201.1 mm to (246.1, 62.7)
- moved R97 191.0 mm to (246.1, 61.2)
- moved C116 187.6 mm to (246.1, 64.2)
- moved R99 186.4 mm to (242.1, 65.9), turned to 90 degrees
- moved C117 185.9 mm to (243.1, 64.2), turned to 180 degrees
- moved C96 180.9 mm to (249.0, 143.4), turned to 90 degrees
- moved U2 176.7 mm to (243.3, 143.7)
- moved R102 175.8 mm to (242.1, 67.7), turned to 90 degrees
- moved TP32 174.8 mm to (248.3, 61.5)
- moved C2 171.4 mm to (247.8, 143.4), turned to -90 degrees
- moved TP33 171.0 mm to (241.7, 60.5)
- moved C190 166.0 mm to (257.2, 48.9), turned to 90 degrees
- moved TP36 165.5 mm to (243.7, 60.6)
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Connections:
- net /+VPGA renamed +5V_PGA
- C10 pad 1: GND -> Net-(IC5B-VD11_1)
- C10 pad 2: +VUSB -> GND
- C1002_1 pad 1: Net-(U1001_1-S3B) -> /OPA_OUT
- C1002_1 pad 2: Net-(U1001_1-S2B) -> /DC_FB
- C1003_1 pad 1: -5V -> -5V_BUF
- C1004_1 pad 2: +5V -> +5V_BUF
- C1005_1 pad 1: -5V -> -5V_BUF
- C1006_1 pad 2: +5V -> +5V_BUF
- C1007_1 pad 1: -5V -> -5V_BUF
- C1008_1 pad 2: +5V -> +5V_BUF
- C1041_1 pad 2: /TRIM -> /TRIM_1
- C1044_1 pad 1: +5V -> +5V_BUF
- C1045_1 pad 1: +5V -> +5V_BUF
- C1046_1 pad 1: +5V -> +5V_BUF
- C1047_1 pad 1: +5V -> +5V_BUF
- C1048_1 pad 1: +5V -> +5V_BUF
- C1049_1 pad 1: +5V -> +5V_BUF
- C1050_1 pad 1: +5V -> +5V_BUF
- C1052_1 pad 2: -5V -> -5V_BUF
- C1053_1 pad 2: -5V -> -5V_BUF
- C1054_1 pad 2: -5V -> -5V_BUF
- C1055_1 pad 2: -5V -> -5V_BUF
- C1056_1 pad 2: -5V -> -5V_BUF
- C1057_1 pad 2: -5V -> -5V_BUF
- C106 pad 2: /-5V_R -> -5V
- C145 pad 2: Net-(IC5B-VA19_1) -> +1V9_ACQ
- C146 pad 2: Net-(IC5B-VPLL19_1) -> +1V1_ACQ
- C147 pad 1: GND -> +3V3
- C147 pad 2: Net-(IC5B-VREFO) -> GND
- C151 pad 2: Net-(IC5B-VA11_10) -> +1V9_ACQ
- C152 pad 2: Net-(IC5B-VD11_10) -> +1V1_ACQ
- C63 pad 1: Net-(IC5B-VA11_10) -> Net-(IC5B-VA11_1)
- C64 pad 1: Net-(IC5B-VA11_10) -> Net-(IC5B-VA11_1)
- C66 pad 1: Net-(IC5B-VA11_10) -> Net-(IC5B-VA11_1)
- C67 pad 1: Net-(IC5B-VA11_10) -> Net-(IC5B-VA11_1)
- C68 pad 1: Net-(IC5B-VD11_10) -> Net-(IC5B-VD11_1)
- C69 pad 1: Net-(IC5B-VD11_10) -> Net-(IC5B-VD11_1)
- C70 pad 1: Net-(IC5B-VD11_10) -> Net-(IC5B-VD11_1)
- C77 pad 1: Net-(IC5B-VD11_10) -> Net-(IC5B-VD11_1)
- C78 pad 1: Net-(IC5B-VD11_10) -> Net-(IC5B-VD11_1)
- FB1001_1 pad 1: /TRIM -> /TRIM_1
- IC1 pad A1: unconnected-(IC1I-GND_1-PadA1) -> GND
- IC1 pad A11: unconnected-(IC1D-DXP_0-PadA11) -> GND
- IC1 pad A12: unconnected-(IC1D-VP_0-PadA12) -> GND
- IC1 pad A13: unconnected-(IC1D-VREFN_0-PadA13) -> GND
- IC1 pad A19: unconnected-(IC1I-GND_6-PadA19) -> GND
- IC1 pad A3: unconnected-(IC1I-GND_2-PadA3) -> GND
- IC1 pad A4: unconnected-(IC1E-MGTPRXN0_216-PadA4) -> /ADC_JESD_0_N
- IC1 pad A5: unconnected-(IC1I-GND_3-PadA5) -> GND
- IC1 pad A6: unconnected-(IC1E-MGTPRXN1_216-PadA6) -> /ADC_JESD_1_N
- IC1 pad A7: unconnected-(IC1I-GND_4-PadA7) -> GND
- IC1 pad A9: unconnected-(IC1I-GND_5-PadA9) -> GND
- IC1 pad B1: unconnected-(IC1F-MGTAVTT_1-PadB1) -> Net-(IC1F-MGTAVTT_1)
- IC1 pad B11: unconnected-(IC1D-DXN_0-PadB11) -> GND
- IC1 pad B12: unconnected-(IC1D-VREFP_0-PadB12) -> GND
- IC1 pad B13: unconnected-(IC1D-VN_0-PadB13) -> GND
- IC1 pad B14: unconnected-(IC1I-GND_11-PadB14) -> GND
- IC1 pad B19: unconnected-(IC1G-VCCO_15_1-PadB19) -> GND
- IC1 pad B3: unconnected-(IC1I-GND_7-PadB3) -> GND
- IC1 pad B4: unconnected-(IC1E-MGTPRXP0_216-PadB4) -> /ADC_JESD_0_P
- IC1 pad B5: unconnected-(IC1I-GND_8-PadB5) -> GND
- IC1 pad B6: unconnected-(IC1E-MGTPRXP1_216-PadB6) -> /ADC_JESD_1_P
- IC1 pad B7: unconnected-(IC1I-GND_9-PadB7) -> GND
- IC1 pad B9: unconnected-(IC1I-GND_10-PadB9) -> GND
- IC1 pad C1: unconnected-(IC1F-MGTAVCC_1-PadC1) -> +1V0_MGT
- IC1 pad C10: unconnected-(IC1I-GND_16-PadC10) -> GND
- IC1 pad C11: unconnected-(IC1D-CCLK_0-PadC11) -> /QSPI_CLK
- IC1 pad C12: unconnected-(IC1I-GNDADC_0-PadC12) -> GND
- IC1 pad C13: unconnected-(IC1H-VCCADC_0-PadC13) -> Net-(IC1H-VCCADC_0)
- IC1 pad C14: unconnected-(IC1G-VCCO_15_2-PadC14) -> GND
- IC1 pad C18: unconnected-(IC1G-VCCO_15_3-PadC18) -> GND
- IC1 pad C19: unconnected-(IC1I-GND_17-PadC19) -> GND
- IC1 pad C2: unconnected-(IC1I-GND_12-PadC2) -> GND
- IC1 pad C3: unconnected-(IC1I-GND_13-PadC3) -> GND
- IC1 pad C4: unconnected-(IC1I-GND_14-PadC4) -> GND
- IC1 pad C5: unconnected-(IC1F-MGTAVTT_2-PadC5) -> Net-(IC1F-MGTAVTT_1)
- IC1 pad C6: unconnected-(IC1I-GND_15-PadC6) -> GND
- IC1 pad C7: unconnected-(IC1E-MGTRREF_216-PadC7) -> Net-(IC1E-MGTRREF_216)
- IC1 pad C8: unconnected-(IC1D-TCK_0-PadC8) -> /TCK
- IC1 pad C9: unconnected-(IC1H-VCCBATT_0-PadC9) -> +1V8
- IC1 pad D17: unconnected-(IC1A-IO_0_14-PadD17) -> Net-(IC1A-IO_0_14)
- IC1 pad D18: unconnected-(IC1A-IO_L1P_T0_D00_MOSI_14-PadD18) -> Net-(IC1A-IO_L1P_T0_D00_MOSI_14)
- IC1 pad D19: unconnected-(IC1A-IO_L1N_T0_D01_DIN_14-PadD19) -> Net-(IC1A-IO_L1N_T0_D01_DIN_14)
- IC1 pad D3: unconnected-(IC1I-GND_18-PadD3) -> GND
- IC1 pad E1: unconnected-(IC1F-MGTAVCC_2-PadE1) -> +1V0_MGT
- IC1 pad E17: unconnected-(IC1A-IO_L3P_T0_DQS_PUDC_B_14-PadE17) -> Net-(IC1A-IO_L3P_T0_DQS_PUDC_B_14)
- IC1 pad E18: unconnected-(IC1A-IO_L3N_T0_DQS_EMCCLK_14-PadE18) -> Net-(IC1A-IO_L3N_T0_DQS_EMCCLK_14)
- IC1 pad E19: unconnected-(IC1A-IO_L2P_T0_D02_14-PadE19) -> Net-(IC1A-IO_L2P_T0_D02_14)
- IC1 pad E2: unconnected-(IC1F-MGTAVTT_3-PadE2) -> Net-(IC1F-MGTAVTT_1)
- IC1 pad E3: unconnected-(IC1I-GND_19-PadE3) -> GND
- IC1 pad F1: unconnected-(IC1I-GND_20-PadF1) -> GND
- IC1 pad F17: unconnected-(IC1A-IO_L5P_T0_D06_14-PadF17) -> Net-(IC1A-IO_L5P_T0_D06_14)
- IC1 pad F18: unconnected-(IC1I-GND_23-PadF18) -> GND
- IC1 pad F19: unconnected-(IC1A-IO_L2N_T0_D03_14-PadF19) -> Net-(IC1A-IO_L2N_T0_D03_14)
- IC1 pad F2: unconnected-(IC1I-GND_21-PadF2) -> GND
- IC1 pad F3: unconnected-(IC1I-GND_22-PadF3) -> GND
- IC1 pad G10: unconnected-(IC1H-VCCINT_1-PadG10) -> +1V0
- IC1 pad G11: unconnected-(IC1I-GND_25-PadG11) -> GND
- IC1 pad G12: unconnected-(IC1G-VCCO_0_1-PadG12) -> +3V3
- IC1 pad G13: unconnected-(IC1G-VCCO_15_4-PadG13) -> GND
- IC1 pad G17: unconnected-(IC1A-IO_L5N_T0_D07_14-PadG17) -> Net-(IC1A-IO_L5N_T0_D07_14)
- IC1 pad G18: unconnected-(IC1A-IO_L4P_T0_D04_14-PadG18) -> Net-(IC1A-IO_L4P_T0_D04_14)
- IC1 pad G19: unconnected-(IC1A-IO_L6P_T0_FCS_B_14-PadG19) -> Net-(IC1A-IO_L6P_T0_FCS_B_14)
- IC1 pad G7: unconnected-(IC1F-MGTAVTT_4-PadG7) -> Net-(IC1F-MGTAVTT_1)
- IC1 pad G8: unconnected-(IC1I-GND_24-PadG8) -> GND
- IC1 pad G9: unconnected-(IC1F-MGTAVCC_3-PadG9) -> +1V0_MGT
- IC1 pad H10: unconnected-(IC1H-VCCINT_2-PadH10) -> +1V0
- IC1 pad H11: unconnected-(IC1I-GND_28-PadH11) -> GND
- IC1 pad H12: unconnected-(IC1I-GND_29-PadH12) -> GND
- IC1 pad H13: unconnected-(IC1H-VCCAUX_1-PadH13) -> +1V8
- IC1 pad H17: unconnected-(IC1A-IO_L7P_T1_D09_14-PadH17) -> Net-(IC1A-IO_L7P_T1_D09_14)
- IC1 pad H18: unconnected-(IC1A-IO_L4N_T0_D05_14-PadH18) -> Net-(IC1A-IO_L4N_T0_D05_14)
- IC1 pad H19: unconnected-(IC1A-IO_L6N_T0_D08_VREF_14-PadH19) -> Net-(IC1A-IO_L6N_T0_D08_VREF_14)
- IC1 pad H7: unconnected-(IC1I-GND_26-PadH7) -> GND
- IC1 pad H8: unconnected-(IC1I-GND_27-PadH8) -> GND
- IC1 pad H9: unconnected-(IC1F-MGTAVCC_4-PadH9) -> +1V0_MGT
- IC1 pad J10: unconnected-(IC1H-VCCINT_3-PadJ10) -> +1V0
- IC1 pad J11: unconnected-(IC1I-GND_33-PadJ11) -> GND
- IC1 pad J12: unconnected-(IC1I-GND_34-PadJ12) -> GND
- IC1 pad J13: unconnected-(IC1H-VCCAUX_2-PadJ13) -> +1V8
- IC1 pad J17: unconnected-(IC1A-IO_L7N_T1_D10_14-PadJ17) -> Net-(IC1A-IO_L7N_T1_D10_14)
- IC1 pad J18: unconnected-(IC1I-GND_35-PadJ18) -> GND
- IC1 pad J19: unconnected-(IC1A-IO_L8P_T1_D11_14-PadJ19) -> Net-(IC1A-IO_L8P_T1_D11_14)
- IC1 pad J2: unconnected-(IC1I-GND_30-PadJ2) -> GND
- IC1 pad J7: unconnected-(IC1G-VCCO_34_1-PadJ7) -> GND
- IC1 pad J8: unconnected-(IC1I-GND_31-PadJ8) -> GND
- IC1 pad J9: unconnected-(IC1I-GND_32-PadJ9) -> GND
- IC1 pad K12: unconnected-(IC1G-VCCO_14_1-PadK12) -> +3V3
- IC1 pad K13: unconnected-(IC1G-VCCO_14_2-PadK13) -> +3V3
- IC1 pad K17: unconnected-(IC1A-IO_L12P_T1_MRCC_14-PadK17) -> Net-(IC1A-IO_L12P_T1_MRCC_14)
- IC1 pad K18: unconnected-(IC1A-IO_L11P_T1_SRCC_14-PadK18) -> Net-(IC1A-IO_L11P_T1_SRCC_14)
- IC1 pad K19: unconnected-(IC1A-IO_L8N_T1_D12_14-PadK19) -> Net-(IC1A-IO_L8N_T1_D12_14)
- IC1 pad K7: unconnected-(IC1G-VCCO_34_2-PadK7) -> GND
- IC1 pad K8: unconnected-(IC1I-GND_36-PadK8) -> GND
- IC1 pad L10: unconnected-(IC1H-VCCINT_4-PadL10) -> +1V0
- IC1 pad L11: unconnected-(IC1I-GND_39-PadL11) -> GND
- IC1 pad L12: unconnected-(IC1G-VCCO_14_3-PadL12) -> +3V3
- IC1 pad L13: unconnected-(IC1G-VCCO_14_4-PadL13) -> +3V3
- IC1 pad L17: unconnected-(IC1A-IO_L12N_T1_MRCC_14-PadL17) -> Net-(IC1A-IO_L12N_T1_MRCC_14)
- IC1 pad L18: unconnected-(IC1A-IO_L11N_T1_SRCC_14-PadL18) -> Net-(IC1A-IO_L11N_T1_SRCC_14)
- IC1 pad L19: unconnected-(IC1A-IO_L9P_T1_DQS_14-PadL19) -> Net-(IC1A-IO_L9P_T1_DQS_14)
- IC1 pad L7: unconnected-(IC1G-VCCO_34_3-PadL7) -> GND
- IC1 pad L8: unconnected-(IC1I-GND_37-PadL8) -> GND
- IC1 pad L9: unconnected-(IC1I-GND_38-PadL9) -> GND
- IC1 pad M10: unconnected-(IC1H-VCCINT_5-PadM10) -> +1V0
- IC1 pad M11: unconnected-(IC1H-VCCBRAM_1-PadM11) -> +1V0
- IC1 pad M12: unconnected-(IC1G-VCCO_14_5-PadM12) -> +3V3
- IC1 pad M13: unconnected-(IC1G-VCCO_14_6-PadM13) -> +3V3
- IC1 pad M17: unconnected-(IC1A-IO_L10P_T1_D14_14-PadM17) -> Net-(IC1A-IO_L10P_T1_D14_14)
- IC1 pad M18: unconnected-(IC1I-GND_42-PadM18) -> GND
- IC1 pad M19: unconnected-(IC1A-IO_L9N_T1_DQS_D13_14-PadM19) -> Net-(IC1A-IO_L9N_T1_DQS_D13_14)
- IC1 pad M2: unconnected-(IC1I-GND_40-PadM2) -> GND
- IC1 pad M7: unconnected-(IC1G-VCCO_34_4-PadM7) -> GND
- IC1 pad M8: unconnected-(IC1G-VCCO_34_5-PadM8) -> GND
- IC1 pad M9: unconnected-(IC1I-GND_41-PadM9) -> GND
- IC1 pad N10: unconnected-(IC1H-VCCINT_6-PadN10) -> +1V0
- IC1 pad N11: unconnected-(IC1H-VCCBRAM_2-PadN11) -> +1V0
- IC1 pad N12: unconnected-(IC1I-GND_44-PadN12) -> GND
- IC1 pad N13: unconnected-(IC1G-VCCO_14_7-PadN13) -> +3V3
- IC1 pad N17: unconnected-(IC1A-IO_L14P_T2_SRCC_14-PadN17) -> Net-(IC1A-IO_L14P_T2_SRCC_14)
- IC1 pad N18: unconnected-(IC1A-IO_L10N_T1_D15_14-PadN18) -> Net-(IC1A-IO_L10N_T1_D15_14)
- IC1 pad N19: unconnected-(IC1A-IO_L13P_T2_MRCC_14-PadN19) -> Net-(IC1A-IO_L13P_T2_MRCC_14)
- IC1 pad N7: unconnected-(IC1G-VCCO_34_6-PadN7) -> GND
- IC1 pad N8: unconnected-(IC1G-VCCO_34_7-PadN8) -> GND
- IC1 pad N9: unconnected-(IC1I-GND_43-PadN9) -> GND
- IC1 pad P18: unconnected-(IC1A-IO_L14N_T2_SRCC_14-PadP18) -> Net-(IC1A-IO_L14N_T2_SRCC_14)
- IC1 pad P19: unconnected-(IC1A-IO_L13N_T2_MRCC_14-PadP19) -> Net-(IC1A-IO_L13N_T2_MRCC_14)
- IC1 pad R18: unconnected-(IC1I-GND_46-PadR18) -> GND
- IC1 pad R19: unconnected-(IC1A-IO_L15P_T2_DQS_RDWR_B_14-PadR19) -> Net-(IC1A-IO_L15P_T2_DQS_RDWR_B_14)
- IC1 pad R2: unconnected-(IC1I-GND_45-PadR2) -> GND
- IC1 pad T19: unconnected-(IC1A-IO_L15N_T2_DQS_DOUT_CSO_B_14-PadT19) -> Net-(IC1A-IO_L15N_T2_DQS_DOUT_CSO_B_14)
- IC1 pad U10: unconnected-(IC1D-PROGRAM_B_0-PadU10) -> Net-(IC1D-PROGRAM_B_0)
- IC1 pad U11: unconnected-(IC1D-DONE_0-PadU11) -> /DONE
- IC1 pad U12: unconnected-(IC1D-CFGBVS_0-PadU12) -> +3V3
- IC1 pad U13: unconnected-(IC1D-M2_0-PadU13) -> /M2
- IC1 pad U19: unconnected-(IC1A-IO_L16P_T2_CSI_B_14-PadU19) -> Net-(IC1A-IO_L16P_T2_CSI_B_14)
- IC1 pad V10: unconnected-(IC1D-TDO_0-PadV10) -> /TDO
- IC1 pad V11: unconnected-(IC1G-VCCO_0_2-PadV11) -> +3V3
- IC1 pad V12: unconnected-(IC1I-GND_50-PadV12) -> GND
- IC1 pad V13: unconnected-(IC1D-M0_0-PadV13) -> /M0
- IC1 pad V15: unconnected-(IC1I-GND_51-PadV15) -> GND
- IC1 pad V18: unconnected-(IC1I-GND_52-PadV18) -> GND
- IC1 pad V19: unconnected-(IC1A-IO_L16N_T2_A15_D31_14-PadV19) -> Net-(IC1A-IO_L16N_T2_A15_D31_14)
- IC1 pad V2: unconnected-(IC1I-GND_47-PadV2) -> GND
- IC1 pad V5: unconnected-(IC1I-GND_48-PadV5) -> GND
- IC1 pad V8: unconnected-(IC1I-GND_49-PadV8) -> GND
- IC1 pad W1: unconnected-(IC1I-GND_53-PadW1) -> GND
- IC1 pad W10: unconnected-(IC1D-TMS_0-PadW10) -> /TMS
- IC1 pad W11: unconnected-(IC1D-TDI_0-PadW11) -> /TDI
- IC1 pad W12: unconnected-(IC1D-INIT_B_0-PadW12) -> Net-(IC1D-INIT_B_0)
- IC1 pad W13: unconnected-(IC1D-M1_0-PadW13) -> /M1
- IC1 pad W19: unconnected-(IC1I-GND_54-PadW19) -> GND
- IC2 pad 40: unconnected-(IC2-DATA_0-Pad40) -> Net-(IC1A-IO_0_14)
- IC2 pad 41: unconnected-(IC2-DATA_1-Pad41) -> Net-(IC1A-IO_L16P_T2_CSI_B_14)
- IC2 pad 42: unconnected-(IC2-DATA_2-Pad42) -> Net-(IC1A-IO_L1N_T0_D01_DIN_14)
- IC2 pad 43: unconnected-(IC2-DATA_3-Pad43) -> Net-(IC1A-IO_L1P_T0_D00_MOSI_14)
- IC2 pad 44: unconnected-(IC2-DATA_4-Pad44) -> Net-(IC1A-IO_L2N_T0_D03_14)
- IC2 pad 45: unconnected-(IC2-DATA_5-Pad45) -> Net-(IC1A-IO_L2P_T0_D02_14)
- IC2 pad 46: unconnected-(IC2-DATA_6-Pad46) -> Net-(IC1A-IO_L3N_T0_DQS_EMCCLK_14)
- IC2 pad 47: unconnected-(IC2-DATA_7-Pad47) -> Net-(IC1A-IO_L3P_T0_DQS_PUDC_B_14)
- IC2 pad 50: unconnected-(IC2-DATA_8-Pad50) -> Net-(IC1A-IO_L4N_T0_D05_14)
- IC2 pad 51: unconnected-(IC2-DATA_9-Pad51) -> Net-(IC1A-IO_L4P_T0_D04_14)
- IC2 pad 52: unconnected-(IC2-DATA_10-Pad52) -> Net-(IC1A-IO_L5N_T0_D07_14)
- IC2 pad 53: unconnected-(IC2-DATA_11-Pad53) -> Net-(IC1A-IO_L5P_T0_D06_14)
- IC2 pad 54: unconnected-(IC2-DATA_12-Pad54) -> Net-(IC1A-IO_L6N_T0_D08_VREF_14)
- IC2 pad 55: unconnected-(IC2-DATA_13-Pad55) -> Net-(IC1A-IO_L6P_T0_FCS_B_14)
- IC2 pad 56: unconnected-(IC2-DATA_14-Pad56) -> Net-(IC1A-IO_L7N_T1_D10_14)
- IC2 pad 57: unconnected-(IC2-DATA_15-Pad57) -> Net-(IC1A-IO_L7P_T1_D09_14)
- IC2 pad 58: unconnected-(IC2-CLK-Pad58) -> Net-(IC1A-IO_L16N_T2_A15_D31_14)
- IC2 pad 60: unconnected-(IC2-DATA_16-Pad60) -> Net-(IC1A-IO_L8N_T1_D12_14)
- IC2 pad 61: unconnected-(IC2-DATA_17-Pad61) -> Net-(IC1A-IO_L8P_T1_D11_14)
- IC2 pad 62: unconnected-(IC2-DATA_18-Pad62) -> Net-(IC1A-IO_L9N_T1_DQS_D13_14)
- IC2 pad 63: unconnected-(IC2-DATA_19-Pad63) -> Net-(IC1A-IO_L9P_T1_DQS_14)
- IC2 pad 64: unconnected-(IC2-DATA_20-Pad64) -> Net-(IC1A-IO_L10N_T1_D15_14)
- IC2 pad 65: unconnected-(IC2-DATA_21-Pad65) -> Net-(IC1A-IO_L10P_T1_D14_14)
- IC2 pad 66: unconnected-(IC2-DATA_22-Pad66) -> Net-(IC1A-IO_L11N_T1_SRCC_14)
- IC2 pad 67: unconnected-(IC2-DATA_23-Pad67) -> Net-(IC1A-IO_L11P_T1_SRCC_14)
- IC2 pad 69: unconnected-(IC2-DATA_24-Pad69) -> Net-(IC1A-IO_L12N_T1_MRCC_14)
- IC2 pad 70: unconnected-(IC2-DATA_25-Pad70) -> Net-(IC1A-IO_L12P_T1_MRCC_14)
- IC2 pad 71: unconnected-(IC2-DATA_26-Pad71) -> Net-(IC1A-IO_L13N_T2_MRCC_14)
- IC2 pad 72: unconnected-(IC2-DATA_27-Pad72) -> Net-(IC1A-IO_L13P_T2_MRCC_14)
- IC2 pad 73: unconnected-(IC2-DATA_28-Pad73) -> Net-(IC1A-IO_L14N_T2_SRCC_14)
- IC2 pad 74: unconnected-(IC2-DATA_29-Pad74) -> Net-(IC1A-IO_L14P_T2_SRCC_14)
- IC2 pad 75: unconnected-(IC2-DATA_30-Pad75) -> Net-(IC1A-IO_L15N_T2_DQS_DOUT_CSO_B_14)
- IC2 pad 76: unconnected-(IC2-DATA_31-Pad76) -> Net-(IC1A-IO_L15P_T2_DQS_RDWR_B_14)
- IC5 pad D5: unconnected-(IC5B-VA19_2-PadD5) -> Net-(IC5B-VA19_1)
- IC5 pad E6: unconnected-(IC5B-VA19_3-PadE6) -> Net-(IC5B-VA19_1)
- IC5 pad E8: unconnected-(IC5A-~{SCS}-PadE8) -> /ADC_SPI_SCS
- IC5 pad F6: unconnected-(IC5B-VA19_4-PadF6) -> Net-(IC5B-VA19_1)
- IC5 pad F8: unconnected-(IC5A-SCLK-PadF8) -> /ADC_SPI_CLK
- IC5 pad G6: unconnected-(IC5B-VA19_5-PadG6) -> Net-(IC5B-VA19_1)
- IC5 pad G8: unconnected-(IC5A-SDI-PadG8) -> /ADC_SPI_SDI
- IC5 pad G9: unconnected-(IC5A-SDO-PadG9) -> /ADC_SPI_SDO
- IC5 pad J6: Net-(IC5B-VA11_10) -> Net-(IC5B-VA11_1)
- IC5 pad M10: Net-(IC5B-VD11_10) -> Net-(IC5B-VD11_1)
- R1003_1 pad 1: Net-(U1001_1-S1B) -> Net-(U1011_1-+)
- R1033_1 pad 1: unconnected-(R1033_1-Pad1) -> +3V3_PGA
- R1036_1 pad 2: -5V -> -5V_BUF
- R1039_1 pad 2: Net-(U1001_1-D1) -> Net-(U1011_1-+)
- R1047_1 pad 1: Net-(U1001_1-D1) -> Net-(U1011_1-+)
- R93 pad 2: /-5V_R -> -5V
- U1009_1 pad 1: +5V -> +5V_BUF
- U1009_1 pad 10: -5V -> -5V_BUF
- U1009_1 pad 12: +5V -> +5V_BUF
- U1009_1 pad 15: +5V -> +5V_BUF
- U1009_1 pad 5: -5V -> -5V_BUF
- U1009_1 pad 6: -5V -> -5V_BUF
- U1009_1 pad 8: -5V -> -5V_BUF
- U1011_1 pad 2: -5V -> -5V_BUF
- U1011_1 pad 3: Net-(U1001_1-S1B) -> Net-(U1011_1-+)
- U1011_1 pad 5: +5V -> +5V_BUF
- U13 pad 4: /-5V_R -> -5V
Routing:
- net Net-(IC1A-IO_L1N_T0_D01_DIN_14): track 0.00 -> 16.0 mm
- net Net-(IC1A-IO_L2P_T0_D02_14): track 0.00 -> 14.9 mm
- net Net-(IC1A-IO_L2N_T0_D03_14): track 0.00 -> 14.5 mm
- net Net-(IC1A-IO_L6P_T0_FCS_B_14): track 0.00 -> 14.4 mm
- net Net-(IC1A-IO_L6N_T0_D08_VREF_14): track 0.00 -> 14.3 mm
- net Net-(IC1A-IO_L8P_T1_D11_14): track 0.00 -> 13.9 mm
- net Net-(IC1A-IO_L7N_T1_D10_14): track 0.00 -> 6.80 mm, vias 0 -> 1
- net Net-(IC1A-IO_L7P_T1_D09_14): track 0.00 -> 5.85 mm, vias 0 -> 1
- net Net-(IC1A-IO_L12P_T1_MRCC_14): track 0.00 -> 5.20 mm, vias 0 -> 1
- net Net-(IC1A-IO_L5N_T0_D07_14): track 0.00 -> 4.90 mm, vias 0 -> 1
- net Net-(IC1A-IO_L12N_T1_MRCC_14): track 0.00 -> 4.01 mm, vias 0 -> 1
- net Net-(IC1A-IO_L5P_T0_D06_14): track 0.00 -> 3.96 mm, vias 0 -> 1
- net Net-(IC1A-IO_L3P_T0_DQS_PUDC_B_14): track 0.00 -> 3.01 mm, vias 0 -> 1
- net Net-(IC1A-IO_L10P_T1_D14_14): track 0.00 -> 2.81 mm, vias 0 -> 1
- net Net-(IC1A-IO_0_14): track 0.00 -> 1.94 mm, vias 0 -> 1
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- added copper zone on F.Cu, net +3V3_PGA
- added copper zone on F.Cu, net +5V
- added copper zone on F.Cu, net /+5V_R_PGA
- added copper zone on In1.Cu, net GND
Other:
- copper layers 2 -> 6

Commit message: m
Parts:
- added C153: 10uF, Passives_SMD:0603_1608Metric, F.Cu at (80.9, 70.3)
- added C156: 10uF, Passives_SMD:0603_1608Metric, F.Cu at (81.5, 55.8)
- added C186: 10uF, Passives_SMD:0603_1608Metric, F.Cu at (61.0, 56.7)
- added C187: 1uF, Passives_SMD:0402_1005Metric, F.Cu at (87.0, 64.5)
- added C188: 1uF, Passives_SMD:0402_1005Metric, F.Cu at (80.9, 57.0)
- added C193: 100nF, Passives_SMD:0402_1005Metric, F.Cu at (83.8, 58.6)
- added C197: 100nF, Passives_SMD:0402_1005Metric, F.Cu at (82.8, 59.0)
- added C198: 100nF, Passives_SMD:0402_1005Metric, F.Cu at (85.1, 67.2)
- added C199: 100nF, Passives_SMD:0402_1005Metric, F.Cu at (89.8, 63.1)
- added C200: 100nF, Passives_SMD:0402_1005Metric, F.Cu at (86.7, 60.8)
- added C201: 1uF, Passives_SMD:0402_1005Metric, F.Cu at (72.7, 64.8)
- added C202: 1uF, Passives_SMD:0402_1005Metric, F.Cu at (84.1, 66.9)
- added C203: 10uF, Passives_SMD:0603_1608Metric, F.Cu at (61.0, 55.2)
- added J1: 10137062-00021LF, Samacsys:1013706200021LF, F.Cu at (102.8, 63.8)
- added J6: 2.54mm 6 Pin TH, Thunderscope_Rev5:GEN_2.54MM_6_PIN_TH_RA, F.Cu at (189.7, 41.2)
- added R15: 1K6R, Passives_SMD:0402_1005Metric, F.Cu at (84.6, 60.7)
- added R16: 4K7R, Passives_SMD:0402_1005Metric, F.Cu at (78.4, 55.5)
- added R17: 10KR, Passives_SMD:0402_1005Metric, F.Cu at (77.4, 54.5)
- added R18: 10KR, Passives_SMD:0402_1005Metric, F.Cu at (85.8, 67.9)
- added R5: DNP (place for LED current limiter), Passives_SMD:0402_1005Metric, F.Cu at (70.0, 73.9)
- added R6: DNP (place for LED), Passives_SMD:0402_1005Metric, F.Cu at (70.0, 74.9)
- added R7: 0, Passives_SMD:0402_1005Metric, F.Cu at (70.0, 72.9)
- added R70: 5.1K, Passives_SMD:0402_1005Metric, F.Cu at (96.5, 64.0)
- added R73: 5.1K, Passives_SMD:0402_1005Metric, F.Cu at (96.5, 63.0)
- added TP58: PCB, Thunderscope_Rev5:GEN_TP_PCB, F.Cu at (87.6, 68.8)
- added TP61: PCB, Thunderscope_Rev5:GEN_TP_PCB, F.Cu at (89.2, 68.0)
- added TP62: PCB, Thunderscope_Rev5:GEN_TP_PCB, F.Cu at (88.7, 66.2)
- added TP67: PCB, Thunderscope_Rev5:GEN_TP_PCB, F.Cu at (73.1, 76.4)
- added Y2: 830107284409, Samacsys:830107284409, F.Cu at (88.4, 61.8)
- C83, C86: moved to F.Cu
- IC2: value FT602Q-B-T -> FT601Q-B-T
- moved J5 62.1 mm to (59.1, 78.2)
- moved R136 50.0 mm to (52.0, 67.2), turned to 180 degrees
- moved R137 49.3 mm to (52.0, 68.2), turned to 180 degrees
- moved C155 43.8 mm to (63.6, 75.8)
- moved S1 42.4 mm to (50.7, 71.5), turned to -90 degrees
- moved C142 32.7 mm to (63.6, 72.0)
- moved C143 32.4 mm to (63.6, 70.5)
- moved C195 31.7 mm to (59.0, 73.6), turned to 180 degrees
- moved U19 30.2 mm to (68.6, 51.8), turned to 180 degrees
- moved C167 29.4 mm to (59.1, 71.9), turned to 180 degrees
- moved C166 25.4 mm to (59.1, 70.4), turned to 180 degrees
- moved F7 24.6 mm to (49.6, 59.2), turned to 180 degrees
- moved F8 24.2 mm to (49.6, 60.6), turned to 180 degrees
- moved C154 24.0 mm to (63.6, 73.8)
- moved C140 23.2 mm to (74.2, 78.3)
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Connections:
- C165 pad 1: +1V0 -> +1V8
- C18 pad 1: Net-(IC1F-MGTAVTT_1) -> +1V2_MGT
- C194 pad 2: AGND -> GND
- C84 pad 1: unconnected-(C84-Pad1) -> +1V2_MGT
- C86 pad 1: unconnected-(C86-Pad1) -> +1V2_MGT
- F8 pad 1: Net-(IC1F-MGTAVTT_1) -> +1V2_MGT
- IC1 pad A14: unconnected-(IC1B-IO_L10P_T1_AD4P_15-PadA14) -> /ADC_SPI_SDI
- IC1 pad A15: unconnected-(IC1B-IO_L10N_T1_AD4N_15-PadA15) -> /ADC_SPI_SCS
- IC1 pad A16: unconnected-(IC1B-IO_L11N_T1_SRCC_AD12N_15-PadA16) -> /ADC_SPI_SDO
- IC1 pad A17: unconnected-(IC1B-IO_L6N_T0_VREF_15-PadA17) -> /ADC_SPI_CLK
- IC1 pad B1: Net-(IC1F-MGTAVTT_1) -> +1V2_MGT
- IC1 pad B19: GND -> +1V8
- IC1 pad C14: GND -> +1V8
- IC1 pad C18: GND -> +1V8
- IC1 pad C5: Net-(IC1F-MGTAVTT_1) -> +1V2_MGT
- IC1 pad D17: Net-(IC1A-IO_0_14) -> /p3
- IC1 pad D18: Net-(IC1A-IO_L1P_T0_D00_MOSI_14) -> /QSPI_DQ0
- IC1 pad D19: Net-(IC1A-IO_L1N_T0_D01_DIN_14) -> /QSPI_DQ1
- IC1 pad E17: Net-(IC1A-IO_L3P_T0_DQS_PUDC_B_14) -> /p2
- IC1 pad E18: Net-(IC1A-IO_L3N_T0_DQS_EMCCLK_14) -> /p9
- IC1 pad E19: Net-(IC1A-IO_L2P_T0_D02_14) -> /QSPI_DQ2
- IC1 pad E2: Net-(IC1F-MGTAVTT_1) -> +1V2_MGT
- IC1 pad F17: Net-(IC1A-IO_L5P_T0_D06_14) -> /p1
- IC1 pad F19: Net-(IC1A-IO_L2N_T0_D03_14) -> /QSPI_DQ3
- IC1 pad G13: GND -> +1V8
- IC1 pad G17: Net-(IC1A-IO_L5N_T0_D07_14) -> /p0
- IC1 pad G18: Net-(IC1A-IO_L4P_T0_D04_14) -> /p10
- IC1 pad G19: Net-(IC1A-IO_L6P_T0_FCS_B_14) -> /QSPI_CS
- IC1 pad G7: Net-(IC1F-MGTAVTT_1) -> +1V2_MGT
- IC1 pad H17: Net-(IC1A-IO_L7P_T1_D09_14) -> /p8
- IC1 pad H18: Net-(IC1A-IO_L4N_T0_D05_14) -> /p11
- IC1 pad H19: Net-(IC1A-IO_L6N_T0_D08_VREF_14) -> /p13
- IC1 pad J17: Net-(IC1A-IO_L7N_T1_D10_14) -> /p7
- IC1 pad J19: Net-(IC1A-IO_L8P_T1_D11_14) -> /p14
- IC1 pad K17: Net-(IC1A-IO_L12P_T1_MRCC_14) -> /p6
- IC1 pad K18: Net-(IC1A-IO_L11P_T1_SRCC_14) -> /p12
- IC1 pad K19: Net-(IC1A-IO_L8N_T1_D12_14) -> /p15
- IC1 pad L17: Net-(IC1A-IO_L12N_T1_MRCC_14) -> /p5
- IC1 pad L18: Net-(IC1A-IO_L11N_T1_SRCC_14) -> /p16
- IC1 pad L19: Net-(IC1A-IO_L9P_T1_DQS_14) -> /p_CLK
- IC1 pad M17: Net-(IC1A-IO_L10P_T1_D14_14) -> /p4
- IC1 pad M19: Net-(IC1A-IO_L9N_T1_DQS_D13_14) -> /p20
- IC1 pad N17: Net-(IC1A-IO_L14P_T2_SRCC_14) -> /BE_3
- IC1 pad N18: Net-(IC1A-IO_L10N_T1_D15_14) -> /p17
- IC1 pad N19: Net-(IC1A-IO_L13P_T2_MRCC_14) -> /p21
- IC1 pad P17: unconnected-(IC1A-IO_L17P_T2_A14_D30_14-PadP17) -> /BE_2
- IC1 pad P18: Net-(IC1A-IO_L14N_T2_SRCC_14) -> /p18
- IC1 pad P19: Net-(IC1A-IO_L13N_T2_MRCC_14) -> /p22
- IC1 pad R17: unconnected-(IC1A-IO_L17N_T2_A13_D29_14-PadR17) -> /BE_0
- IC1 pad R19: Net-(IC1A-IO_L15P_T2_DQS_RDWR_B_14) -> /p23
- IC1 pad T17: unconnected-(IC1A-IO_L18P_T2_A12_D28_14-PadT17) -> /BE_1
- IC1 pad T18: unconnected-(IC1A-IO_L18N_T2_A11_D27_14-PadT18) -> /p19
- IC1 pad T19: Net-(IC1A-IO_L15N_T2_DQS_DOUT_CSO_B_14) -> /p24
- IC1 pad U14: unconnected-(IC1A-IO_25_14-PadU14) -> /WR_N
- IC1 pad U15: unconnected-(IC1A-IO_L22P_T3_A05_D21_14-PadU15) -> /TXE_N
- IC1 pad U16: unconnected-(IC1A-IO_L22N_T3_A04_D20_14-PadU16) -> /RD_N
- IC1 pad U17: unconnected-(IC1A-IO_L19P_T3_A10_D26_14-PadU17) -> /OE_N
- IC1 pad U19: Net-(IC1A-IO_L16P_T2_CSI_B_14) -> /p25
- IC1 pad V14: unconnected-(IC1A-IO_L23P_T3_A03_D19_14-PadV14) -> /SIWU_N
- IC1 pad V16: unconnected-(IC1A-IO_L21P_T3_DQS_14-PadV16) -> /RXF_N
- IC1 pad V19: Net-(IC1A-IO_L16N_T2_A15_D31_14) -> /p26
- IC1 pad W14: unconnected-(IC1A-IO_L23N_T3_A02_D18_14-PadW14) -> /p31_FPGA
- IC1 pad W15: unconnected-(IC1A-IO_L24P_T3_A01_D17_14-PadW15) -> /p30
- IC1 pad W16: unconnected-(IC1A-IO_L24N_T3_A00_D16_14-PadW16) -> /p29
- IC1 pad W17: unconnected-(IC1A-IO_L20P_T3_A08_D24_14-PadW17) -> /p28
- IC1 pad W18: unconnected-(IC1A-IO_L20N_T3_A07_D23_14-PadW18) -> /p27
- IC2 pad 1: unconnected-(IC2B-GND_1-Pad1) -> GND
- IC2 pad 10: unconnected-(IC2C-RESERVED1-Pad10) -> /SIWU_N
- IC2 pad 11: unconnected-(IC2C-WR_N-Pad11) -> /WR_N
- IC2 pad 12: unconnected-(IC2C-RESERVED2-Pad12) -> /RD_N
- IC2 pad 13: unconnected-(IC2C-RESERVED3-Pad13) -> /OE_N
- IC2 pad 14: unconnected-(IC2B-VCCIO_1-Pad14) -> +3V3
- IC2 pad 15: unconnected-(IC2C-RESET_N-Pad15) -> Net-(IC2C-RESET_N)
- IC2 pad 16: unconnected-(IC2C-INT_N-Pad16) -> Net-(IC2C-WAKEUP_N)
- IC2 pad 17: unconnected-(IC2C-SCL-Pad17) -> Net-(IC2C-GPIO0)
- IC2 pad 18: unconnected-(IC2C-SDA-Pad18) -> Net-(IC2C-GPIO1)
- IC2 pad 2: unconnected-(IC2B-AVDD-Pad2) -> Net-(IC2B-AVDD)
- IC2 pad 20: unconnected-(IC2B-VCC33_1-Pad20) -> +3V3
- IC2 pad 21: unconnected-(IC2C-XI-Pad21) -> /FTDI_XI
- IC2 pad 22: unconnected-(IC2C-XO-Pad22) -> /FTDI_XO
- IC2 pad 23: unconnected-(IC2C-DP-Pad23) -> /DP
- IC2 pad 24: unconnected-(IC2B-VCC33_2-Pad24) -> +3V3
- IC2 pad 25: unconnected-(IC2C-DM-Pad25) -> /DN
- IC2 pad 26: unconnected-(IC2B-GND_2-Pad26) -> GND
- IC2 pad 27: unconnected-(IC2C-RREF-Pad27) -> Net-(IC2C-RREF)
- IC2 pad 28: unconnected-(IC2B-VDDA-Pad28) -> +3V3
- IC2 pad 29: unconnected-(IC2B-GND_3-Pad29) -> GND
- IC2 pad 3: unconnected-(IC2B-VD10_1-Pad3) -> Net-(IC2B-AVDD)
- IC2 pad 30: unconnected-(IC2B-VD10_2-Pad30) -> Net-(IC2B-AVDD)
- IC2 pad 31: unconnected-(IC2C-TODN-Pad31) -> Net-(IC2C-TODN)
- IC2 pad 32: unconnected-(IC2C-TODP-Pad32) -> Net-(IC2C-TODP)
- IC2 pad 33: unconnected-(IC2B-VD10_3-Pad33) -> Net-(IC2B-AVDD)
- IC2 pad 34: unconnected-(IC2C-RIDN-Pad34) -> /SSRXN
- IC2 pad 35: unconnected-(IC2C-RIDP-Pad35) -> /SSRXP
- IC2 pad 36: unconnected-(IC2B-GND_4-Pad36) -> GND
- IC2 pad 37: unconnected-(IC2B-VBUS-Pad37) -> Net-(IC2B-VBUS)
- IC2 pad 38: unconnected-(IC2B-VCC33_3-Pad38) -> +3V3
- IC2 pad 39: unconnected-(IC2B-VD10_4-Pad39) -> Net-(IC2B-AVDD)
- IC2 pad 4: unconnected-(IC2C-BE_0-Pad4) -> /BE_0
- IC2 pad 40: Net-(IC1A-IO_0_14) -> /p0
- IC2 pad 41: Net-(IC1A-IO_L16P_T2_CSI_B_14) -> /p1
- IC2 pad 42: Net-(IC1A-IO_L1N_T0_D01_DIN_14) -> /p2
- IC2 pad 43: Net-(IC1A-IO_L1P_T0_D00_MOSI_14) -> /p3
- IC2 pad 44: Net-(IC1A-IO_L2N_T0_D03_14) -> /p4
- IC2 pad 45: Net-(IC1A-IO_L2P_T0_D02_14) -> /p5
- IC2 pad 46: Net-(IC1A-IO_L3N_T0_DQS_EMCCLK_14) -> /p6
- IC2 pad 47: Net-(IC1A-IO_L3P_T0_DQS_PUDC_B_14) -> /p7
- IC2 pad 48: unconnected-(IC2B-VD10_5-Pad48) -> Net-(IC2B-AVDD)
- IC2 pad 49: unconnected-(IC2B-VCCIO_2-Pad49) -> +3V3
- IC2 pad 5: unconnected-(IC2C-BE_1-Pad5) -> /BE_1
- IC2 pad 50: Net-(IC1A-IO_L4N_T0_D05_14) -> /p8
- IC2 pad 51: Net-(IC1A-IO_L4P_T0_D04_14) -> /p9
- IC2 pad 52: Net-(IC1A-IO_L5N_T0_D07_14) -> /p10
- IC2 pad 53: Net-(IC1A-IO_L5P_T0_D06_14) -> /p11
- IC2 pad 54: Net-(IC1A-IO_L6N_T0_D08_VREF_14) -> /p12
- IC2 pad 55: Net-(IC1A-IO_L6P_T0_FCS_B_14) -> /p13
- IC2 pad 56: Net-(IC1A-IO_L7N_T1_D10_14) -> /p14
- IC2 pad 57: Net-(IC1A-IO_L7P_T1_D09_14) -> /p15
- IC2 pad 58: Net-(IC1A-IO_L16N_T2_A15_D31_14) -> /p_CLK
- IC2 pad 59: unconnected-(IC2B-VCCIO_3-Pad59) -> +3V3
- IC2 pad 6: unconnected-(IC2C-BE_2-Pad6) -> /BE_2
- IC2 pad 60: Net-(IC1A-IO_L8N_T1_D12_14) -> /p16
- IC2 pad 61: Net-(IC1A-IO_L8P_T1_D11_14) -> /p17
- IC2 pad 62: Net-(IC1A-IO_L9N_T1_DQS_D13_14) -> /p18
- IC2 pad 63: Net-(IC1A-IO_L9P_T1_DQS_14) -> /p19
- IC2 pad 64: Net-(IC1A-IO_L10N_T1_D15_14) -> /p20
- IC2 pad 65: Net-(IC1A-IO_L10P_T1_D14_14) -> /p21
- IC2 pad 66: Net-(IC1A-IO_L11N_T1_SRCC_14) -> /p22
- IC2 pad 67: Net-(IC1A-IO_L11P_T1_SRCC_14) -> /p23
- IC2 pad 68: unconnected-(IC2B-VCCIO_4-Pad68) -> +3V3
- IC2 pad 69: Net-(IC1A-IO_L12N_T1_MRCC_14) -> /p24
- IC2 pad 7: unconnected-(IC2C-BE_3-Pad7) -> /BE_3
- IC2 pad 70: Net-(IC1A-IO_L12P_T1_MRCC_14) -> /p25
- IC2 pad 71: Net-(IC1A-IO_L13N_T2_MRCC_14) -> /p26
- IC2 pad 72: Net-(IC1A-IO_L13P_T2_MRCC_14) -> /p27
- IC2 pad 73: Net-(IC1A-IO_L14N_T2_SRCC_14) -> /p28
- IC2 pad 74: Net-(IC1A-IO_L14P_T2_SRCC_14) -> /p29
- IC2 pad 75: Net-(IC1A-IO_L15N_T2_DQS_DOUT_CSO_B_14) -> /p30
- IC2 pad 76: Net-(IC1A-IO_L15P_T2_DQS_RDWR_B_14) -> /p31
- IC2 pad 77: unconnected-(IC2B-EP-Pad77) -> GND
- IC2 pad 8: unconnected-(IC2C-TXE_N-Pad8) -> /TXE_N
- IC2 pad 9: unconnected-(IC2C-RXF_N-Pad9) -> /RXF_N
Routing:
- net /BE_3: track 0.00 -> 32.7 mm, vias 0 -> 2
- net /BE_2: track 0.00 -> 29.7 mm, vias 0 -> 2
- net /SIWU_N: track 0.00 -> 29.3 mm, vias 0 -> 2
- net +VUSB: track 0.00 -> 28.7 mm, vias 0 -> 3
- net /BE_1: track 0.00 -> 28.4 mm, vias 0 -> 2
- net /RXF_N: track 0.00 -> 27.2 mm, vias 0 -> 2
- net /TXE_N: track 0.00 -> 25.9 mm, vias 0 -> 2
- net /OE_N: track 0.00 -> 25.2 mm, vias 0 -> 2
- net /RD_N: track 0.00 -> 24.9 mm, vias 0 -> 2
- net /BE_0: track 0.00 -> 24.9 mm, vias 0 -> 2
- net /p4: track 0.00 -> 23.5 mm, vias 0 -> 2
- net /WR_N: track 0.00 -> 23.0 mm, vias 0 -> 2
- net /p0: track 0.00 -> 21.9 mm, vias 0 -> 2
- net /p5: track 0.00 -> 21.2 mm, vias 0 -> 2
- net /p6: track 0.00 -> 20.3 mm, vias 0 -> 2
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- added copper zone on F.Cu, net +1V0_MGT
- added copper zone on In2.Cu, net +1V0_MGT
- added copper zone on F.Cu, net +1V2_MGT
- added copper zone on In2.Cu, net +1V2_MGT
- added copper zone on B.Cu, net +3V3
- added copper zone on F.Cu, net +3V3
- added copper zone on In4.Cu, net GND
Other:
- board text added: "stackup: JLC06161H-3313"
