File: oscillogoat_0.1.kicad_sch (KiCad schematic)
At the start: 342 parts, among them IC1 XC7A12T-1CPG238C, IC2 FT602Q-B-T, IC5 ADC09DJ800AAV, J1002_1 BNC, J3_1 UFL, J4_1 UFL, J5 2.54mm 6 Pin TH, Q1 DMN62D0UW, Q2 DMN62D0UW, U1001_1 TMUX4053, U1008_1 LMH6518, U1009_1 BUF802, U1011_1 OPA140AIDBVR, U13 LM27761, U14 TPS7A9101, U15 TPS7A9101, U16 TPS7A2033, U17 TPS61023, U18 TPS7A9101, U19 MX25L6433FZNI-08G, U2 MCP4452-104E, U20 TPS62A02, U21 TPS62A02, U22 TPS7A9101, U24 TPS62A02, U3 MCP4728, U4 REF2025, U5 OPA140AIDBVR, U8 TPS62A02, Y1 ASEMPLV-100.000MHZ-LR-T

Commit message: update
Parts:
- removed C1001_1: 100pF, Thunderscope_Rev5:GEN_C_0402, symbol Thunderscope_Rev5:CAP 100pF 50V C0G 0402
- removed C103, C1036_1, C1037_1, C141, C193, C61, C65, C79: 1uF, Thunderscope_Rev5:GEN_C_0402, symbol Thunderscope_Rev5:CAP 1uF 25V X5R 0402
- removed C1031_1: 10nF, Thunderscope_Rev5:GEN_C_0603, symbol Thunderscope_Rev5:CAP 10nF 50V C0G 0603
- removed C1039_1, C147, C153, C197, C204: 10uF, Thunderscope_Rev5:GEN_C_0603, symbol Thunderscope_Rev5:CAP 10uF 25V X5R 0603
- removed C97, C98: 22uF, Thunderscope_Rev5:GEN_C_0805, symbol Thunderscope_Rev5:CAP 22uF 25V X5R 0805
- removed FB1000_1, R91: 120@100MHZ, Thunderscope_Rev5:GEN_R_0402, symbol Thunderscope_Rev5:FERRITE BEAD 120 OHM 0402
- removed J3_1, J4_1: UFL, Thunderscope_Rev5:TE_2334884-1, symbol Thunderscope_Rev5:UFL Jack SMD
- removed R101, R108, R114, R115, R133, R135, R142, R144: 0R1, Thunderscope_Rev5:GEN_R_0402, symbol Thunderscope_Rev5:RES 4.7K OHM 1% 1/10W 0402
- removed R1052_1: 10K, Thunderscope_Rev5:GEN_R_0402, symbol Thunderscope_Rev5:RES 10K OHM 1% 1/10W 0402
- removed S1: 416131160803, 416131160803:416131160803, symbol manually_imported:416131160803
- removed TP1016_1, TP1018_1, TP29, TP31, TP35, TP39, TP4: PCB, Thunderscope_Rev5:GEN_TP_PCB, symbol Thunderscope_Rev5:TP PCB 1mm
- removed U1001_1: TMUX4053, Thunderscope_Rev5:TI_TSOT-23-16_DYY0016A, symbol Thunderscope_Rev5:IC SWITCH 3X SPDT TMUX4053
- added C1, C10, C13, C14, C15, C16, C17, C18, C19, C20, C21: 100u, Passives_SMD:1206_3216Metric, symbol manually_created:capacitor_ceramic
- added C1007_2, C1007_3, C1008_2: 10uF, Passives_SMD:0603_1608Metric, symbol Thunderscope_Rev5:CAP 10uF 25V X5R 0603
- added C147: 1uF, Passives_SMD:0402_1005Metric, symbol Thunderscope_Rev5:CAP 1uF 25V X5R 0402
- added F1, F10, F11, F2, F3, F4, F5, F6, F7, F8, F9: 120@100MHZ, Passives_SMD:0402_1005Metric, symbol Thunderscope_Rev5:FERRITE BEAD 120 OHM 0402
- added S1: 416131160803, Snapeda:416131160803, symbol Snapeda:416131160803
- C100, C1002_1, C1032_1, C1033_1, C1034_1, C1035_1, C1041_1, C1042_1, C123, C124, C129, C132, C174, C178, C185, C190, C4, C74, C82: footprint Thunderscope_Rev5:GEN_C_0402 -> Passives_SMD:0402_1005Metric
- C1003_1, C1004_1, C1005_1, C1006_1, C1007_1, C1008_1, C1040_1, C106, C111, C114, C115, C116, C117, C119, C12, C120, C121, C122, C130, C131, C133, C142, C143, C144, C145, C146, C148, C149, C150, C151, C152, C166, C167, C169, C170, C175, C179, C181, C182, C183, C184, C189, C71, C72, C73, C85, C9, C93, C94, C95, C96: footprint Thunderscope_Rev5:GEN_C_0603 -> Passives_SMD:0603_1608Metric; TYPE_SERIAL (none) -> 5
- C101, C104, C105, C128, C154, C155, C168, C176, C177, C180, C191, C195, C75, C99: footprint Thunderscope_Rev5:GEN_C_0805 -> Passives_SMD:0805_2012Metric
- C102, C1038_1, C1043_1, C1044_1, C1045_1, C1046_1, C1047_1, C1048_1, C1049_1, C1050_1, C1052_1, C1053_1, C1054_1, C1055_1, C1056_1, C1057_1, C11, C112, C125, C126, C127, C138, C139, C140, C163, C164, C165, C171, C172, C173, C192, C194, C196, C2, C3, C5, C55, C56, C57, C58, C59, C6, C60, C62, C63, C64, C66, C67, C68, C69, C7, C70, C76, C77, C78, C8, C80, C81, C83, C84, C86: footprint Thunderscope_Rev5:GEN_C_0402 -> Passives_SMD:0402_1005Metric; TYPE_SERIAL (none) -> 2
- C1030_1: footprint Thunderscope_Rev5:GEN_C_0603 -> Passives_SMD:0603_1608Metric
- FB1001_1, R1, R10, R100, R102, R1033_1, R1036_1, R1037_1, R1039_1, R104, R1041_1, R1042_1, R1043_1, R1044_1, R1045_1, R1046_1, R1047_1, R1048_1, R105, R106, R107, R109, R11, R110, R111, R112, R113, R117, R118, R119, R12, R121, R122, R124, R125, R127, R131, R132, R136, R137, R138, R139, R140, R141, R143, R3, R4, R52_1, R55, R56, R66, R67, R68, R69, R71, R72, R9, R90, R93, R96, R97_1, R99: footprint Thunderscope_Rev5:GEN_R_0402 -> Passives_SMD:0402_1005Metric
- L1, L2, L3, L5, L6: footprint Thunderscope_Rev5:GEN_L_1210 -> Passives_SMD:1210_3225Metric
- R1003_1, R1022_1, R1035_1, R1038_1: footprint Thunderscope_Rev5:GEN_R_0603 -> Passives_SMD:0603_1608Metric
- R103, R116, R120, R123, R134, R14, R57, R97, R98: value 0.01 -> 0R01; footprint Thunderscope_Rev5:GEN_R_0603 -> Passives_SMD:0603_1608Metric
Connections:
- net -5V_R is gone; now on net -5V: C106.2, R93.2, U13.4 (VOUT)
- net TRIM is gone; now on net TRIM_1: C1041_1.2, FB1001_1.1
- net +1V0: now also F7.2
- net +1V0_MGT: now also C17.1, F7.1
- net +1V1_ACQ: now also C146.2, C152.2, F1.2, F2.2, F3.2
- net +1V2_MGT: now also F8.2
- net +1V9_ACQ: now also C145.2, C151.2, F4.2, F5.2, F6.2
- net +3V3: now also C147.1
- net +3V3_PGA: now also R1033_1.1
- net +5V: now also C1007_3.1, F11.2, F9.1; no longer C1004_1.2, C1006_1.2, C1008_1.2, C1044_1.1, C1045_1.1, C1046_1.1, C1047_1.1, C1048_1.1, C1049_1.1, C1050_1.1, U1009_1.1 (Vs+), U1009_1.12 (Vso+), U1009_1.15 (CLH), U1011_1.5 (V+)
- net -5V: now also C1007_2.1, F10.1; no longer C1003_1.1, C1005_1.1, C1007_1.1, C1052_1.2, C1053_1.2, C1054_1.2, C1055_1.2, C1056_1.2, C1057_1.2, R1036_1.2, U1009_1.10 (Vso-), U1009_1.5 (Vs-), U1009_1.6 (Aux_Bias), U1009_1.8 (Vs-), U1011_1.2 (V-)
- net DC_FB: now also C1002_1.2
- net GND: now also C1.2, C10.2, C1007_2.2, C1007_3.2, C1008_2.1, C13.2, C14.2, C147.2, C15.2, C16.2, C17.2, C18.2, C19.2, C20.2, C21.2, S1.1, S1.2, S1.3
- net M0: now also S1.A3
- net M1: now also S1.A2
- net M2: now also S1.A1
- net OPA_OUT: now also C1002_1.1
- net at C80.1, IC5.J8 (VTRIG_1), IC5.K8 (VTRIG_2): now also C1.1, F1.1
- net at R1039_1.2, R1047_1.1: now also R1003_1.1, U1011_1.3 (+)
- net at C62.1, IC5.K6 (VREFO): now also C15.1, F5.1
- net at IC2.41 (DATA_1): now also IC1.U19 (IO_L16P_T2_CSI_B_14); no longer IC1.U14 (IO_25_14)
- net at C63.1, C64.1, C66.1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: now also C13.1, F3.1; no longer C151.2
- net at C57.1, C58.1, C59.1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: now also C14.1, F4.1; no longer C145.2
- net at IC1.B1 (MGTAVTT_1), IC1.C5 (MGTAVTT_2), IC1.E2 (MGTAVTT_3)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: now also C18.1, F8.1
- net at C68.1, C69.1, C70.1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: now also C10.1, F2.1; no longer C152.2
- net at C55.1, C56.1, IC5.J4 (VPLL19_1)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: now also C16.1, F6.1; no longer C146.2
- net at IC1.V19 (IO_L16N_T2_A15_D31_14): now also IC2.58 (CLK)
- net +VPGA renamed +5V_PGA
- net +5V_PGA: now also C1008_2.2, C19.1, F9.2
- new net +5V_BUF: C1004_1.2, C1006_1.2, C1008_1.2, C1044_1.1, C1045_1.1, C1046_1.1, C1047_1.1, C1048_1.1, C1049_1.1, C1050_1.1, C21.1, F11.1, U1009_1.1 (Vs+), U1009_1.12 (Vso+), U1009_1.15 (CLH), U1011_1.5 (V+)
- new net -5V_BUF: C1003_1.1, C1005_1.1, C1007_1.1, C1052_1.2, C1053_1.2, C1054_1.2, C1055_1.2, C1056_1.2, C1057_1.2, C20.1, F10.2, R1036_1.2, U1009_1.10 (Vso-), U1009_1.5 (Vs-), U1009_1.6 (Aux_Bias), U1009_1.8 (Vs-), U1011_1.2 (V-)
- no-connect marks 110 -> 109
Other:
- note added: "FPGA IO and USB"
- note removed: "FPGA to USB"
- note removed: "Front End Voltage Regulators"
- note removed: "This cap is switched in during AC coupling"
- note removed: "This cap is switched in during DC coupling"
- moved on the sheet: C100, C1003_1, C1004_1, C1005_1, C1006_1, C1007_1, C1008_1, C101, C102, C1030_1, C1032_1, C1033_1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

Commit message: m
Parts:
- removed IC2: FT602Q-B-T, Samacsys:QFN40P900X900X100-77N-D, symbol Samacsys:FT602Q-B-T
- added C153, C156, C186, C203: 10uF, Passives_SMD:0603_1608Metric, symbol Thunderscope_Rev5:CAP 10uF 25V X5R 0603
- added C187, C188, C201, C202: 1uF, Passives_SMD:0402_1005Metric, symbol Thunderscope_Rev5:CAP 1uF 25V X5R 0402
- added C193, C197, C198, C199, C200: 100nF, Passives_SMD:0402_1005Metric, symbol Thunderscope_Rev5:CAP 1uF 25V X5R 0402
- added IC2: FT601Q-B-T, Samacsys:QFN40P900X900X100-77N-D, symbol Samacsys:FT601Q-B-T
- added J1: 10137062-00021LF, Samacsys:1013706200021LF, symbol Samacsys:10137062-00021LF
- added J6: 2.54mm 6 Pin TH, Thunderscope_Rev5:GEN_2.54MM_6_PIN_TH_RA, symbol Thunderscope_Rev5:CONN 2.54mm 6 Pin TH RA
- added R15: 1K6R, Passives_SMD:0402_1005Metric, symbol Thunderscope_Rev5:RES 0.01 OHM 1% 1/4W 0603
- added R16: 4K7R, Passives_SMD:0402_1005Metric, symbol Thunderscope_Rev5:RES 0.01 OHM 1% 1/4W 0603
- added R17, R18: 10KR, Passives_SMD:0402_1005Metric, symbol Thunderscope_Rev5:RES 0.01 OHM 1% 1/4W 0603
- added R5: DNP (place for LED current limiter), Passives_SMD:0402_1005Metric, symbol Thunderscope_Rev5:RES DNP 0402
- added R6: DNP (place for LED), Passives_SMD:0402_1005Metric, symbol Thunderscope_Rev5:RES DNP 0402
- added R7: 0, Passives_SMD:0402_1005Metric, symbol Thunderscope_Rev5:RES DNP 0402
- added R70, R73: 5.1K, Passives_SMD:0402_1005Metric, symbol Thunderscope_Rev5:RES 10K OHM 1% 1/10W 0402
- added TP58, TP61, TP62, TP67: PCB, Thunderscope_Rev5:GEN_TP_PCB, symbol Thunderscope_Rev5:TP PCB 1mm
- added Y2: 830107284409, Samacsys:830107284409, symbol Samacsys:830107284409
Connections:
- net AGND is gone; now on net GND: C194.2
- net +1V0: no longer C165.1
- net +1V2_MGT: now also C18.1, C84.1, C86.1, F8.1, IC1.B1 (MGTAVTT_1), IC1.C5 (MGTAVTT_2), IC1.E2 (MGTAVTT_3), IC1.G7 (MGTAVTT_4)
- net +1V8: now also C165.1, IC1.B19 (VCCO_15_1), IC1.C14 (VCCO_15_2), IC1.C18 (VCCO_15_3), IC1.G13 (VCCO_15_4), C186.2, C203.2
- net +1V9_ACQ: now also J6.1
- net +3V3: now also C156.2, C187.1, C188.1, C201.1, C202.1, IC2.14 (VCCIO_1), IC2.20 (VCC33_1), IC2.24 (VCC33_2), IC2.28 (VDDA), IC2.38 (VCC33_3), IC2.49 (VCCIO_2), IC2.59 (VCCIO_3), IC2.68 (VCCIO_4), R18.1
- net +VUSB: now also J1.A4 (VBUS_1), J1.A9 (VBUS_2), J1.B4 (VBUS_3), J1.B9 (VBUS_4), R16.2
- net ADC_SPI_CLK: now also IC1.A17 (IO_L6N_T0_VREF_15), J6.2
- net ADC_SPI_SCS: now also IC1.A15 (IO_L10N_T1_AD4N_15), J6.3
- net ADC_SPI_SDI: now also IC1.A14 (IO_L10P_T1_AD4P_15), J6.4
- net ADC_SPI_SDO: now also IC1.A16 (IO_L11N_T1_SRCC_AD12N_15), J6.5
- net GND: now also C153.1, C156.1, C186.1, C187.2, C188.2, C198.1, C199.1, C200.2, C201.2, C202.2, C203.1, IC2.1 (GND_1), IC2.26 (GND_2), IC2.29 (GND_3), IC2.36 (GND_4), IC2.77 (THERMAL_PAD), J1.A1 (GND_1), J1.A12 (GND_2), J1.B1 (GND_3), J1.B12 (GND_4), J1.MH3 (MH4), J1.MH4 (MH1), J1.MH5 (MH3), J1.MH6 (MH2), J6.6, R15.1, R17.1, R6.1, R70.1, R73.2, Y2.2 (GND_1), Y2.4 (GND_2); no longer IC1.B19 (VCCO_15_1), IC1.C14 (VCCO_15_2), IC1.C18 (VCCO_15_3), IC1.G13 (VCCO_15_4)
- net QSPI_CS: now also IC1.G19 (IO_L6P_T0_FCS_B_14)
- net QSPI_DQ0: now also IC1.D18 (IO_L1P_T0_D00_MOSI_14)
- net QSPI_DQ1: now also IC1.D19 (IO_L1N_T0_D01_DIN_14)
- net QSPI_DQ2: now also IC1.E19 (IO_L2P_T0_D02_14)
- net QSPI_DQ3: now also IC1.F19 (IO_L2N_T0_D03_14)
- net p3: now reaches IC1.D17 (IO_0_14)
- net p3: now also IC2.43 (DATA_3)
- net p25: now reaches IC1.U19 (IO_L16P_T2_CSI_B_14)
- net p25: now also IC2.70 (DATA_25)
- net p9: now reaches IC1.E18 (IO_L3N_T0_DQS_EMCCLK_14)
- net p9: now also IC2.51 (DATA_9)
- net p2: now reaches IC1.E17 (IO_L3P_T0_DQS_PUDC_B_14)
- net p2: now also IC2.42 (DATA_2)
- net p11: now reaches IC1.H18 (IO_L4N_T0_D05_14)
- net p11: now also IC2.53 (DATA_11)
- net p10: now reaches IC1.G18 (IO_L4P_T0_D04_14)
- net p10: now also IC2.52 (DATA_10)
- net p0: now reaches IC1.G17 (IO_L5N_T0_D07_14)
- net p0: now also IC2.40 (DATA_0)
- net p1: now reaches IC1.F17 (IO_L5P_T0_D06_14)
- net p1: now also IC2.41 (DATA_1)
- net p13: now reaches IC1.H19 (IO_L6N_T0_D08_VREF_14)
- net p13: now also IC2.55 (DATA_13)
- net p7: now reaches IC1.J17 (IO_L7N_T1_D10_14)
- net p7: now also IC2.47 (DATA_7)
- net p8: now reaches IC1.H17 (IO_L7P_T1_D09_14)
- net p8: now also IC2.50 (DATA_8)
- net p26: now reaches IC1.V19 (IO_L16N_T2_A15_D31_14)
- net p26: now also IC2.71 (DATA_26)
- net p15: now reaches IC1.K19 (IO_L8N_T1_D12_14)
- net p15: now also IC2.57 (DATA_15)
- net p14: now reaches IC1.J19 (IO_L8P_T1_D11_14)
- net p14: now also IC2.56 (DATA_14)
- net p20: now reaches IC1.M19 (IO_L9N_T1_DQS_D13_14)
- net p20: now also IC2.64 (DATA_20)
- net p_CLK: now reaches IC1.L19 (IO_L9P_T1_DQS_14)
- net p_CLK: now also IC2.58 (CLK)
- net p17: now reaches IC1.N18 (IO_L10N_T1_D15_14)
- net p17: now also IC2.61 (DATA_17)
- net p4: now reaches IC1.M17 (IO_L10P_T1_D14_14)
- net p4: now also IC2.44 (DATA_4)
- net p16: now reaches IC1.L18 (IO_L11N_T1_SRCC_14)
- net p16: now also IC2.60 (DATA_16)
- net p12: now reaches IC1.K18 (IO_L11P_T1_SRCC_14)
- net p12: now also IC2.54 (DATA_12)
- net p5: now reaches IC1.L17 (IO_L12N_T1_MRCC_14)
- net p5: now also IC2.45 (DATA_5)
- net p6: now reaches IC1.K17 (IO_L12P_T1_MRCC_14)
- net p6: now also IC2.46 (DATA_6)
- net p22: now reaches IC1.P19 (IO_L13N_T2_MRCC_14)
- net p22: now also IC2.66 (DATA_22)
- net p21: now reaches IC1.N19 (IO_L13P_T2_MRCC_14)
- net p21: now also IC2.65 (DATA_21)
- net p18: now reaches IC1.P18 (IO_L14N_T2_SRCC_14)
- net p18: now also IC2.62 (DATA_18)
- net BE_3: now reaches IC1.N17 (IO_L14P_T2_SRCC_14)
- net BE_3: now also IC2.7 (BE_3)
- net p24: now reaches IC1.T19 (IO_L15N_T2_DQS_DOUT_CSO_B_14)
- net p24: now also IC2.69 (DATA_24)
- net p23: now reaches IC1.R19 (IO_L15P_T2_DQS_RDWR_B_14)
- net p23: now also IC2.67 (DATA_23)
- net BE_2: now reaches IC1.P17 (IO_L17P_T2_A14_D30_14)
- net BE_2: now also IC2.6 (BE_2)
- net BE_0: now reaches IC1.R17 (IO_L17N_T2_A13_D29_14)
- net BE_0: now also IC2.4 (BE_0)
- net BE_1: now reaches IC1.T17 (IO_L18P_T2_A12_D28_14)
- net BE_1: now also IC2.5 (BE_1)
- net p19: now reaches IC1.T18 (IO_L18N_T2_A11_D27_14)
- net p19: now also IC2.63 (DATA_19)
- net WR_N: now reaches IC1.U14 (IO_25_14)
- net WR_N: now also IC2.11 (WR_N)
- net TXE_N: now reaches IC1.U15 (IO_L22P_T3_A05_D21_14)
- net TXE_N: now also IC2.8 (TXE_N)
- net RD_N: now reaches IC1.U16 (IO_L22N_T3_A04_D20_14)
- net RD_N: now also IC2.12 (RD_N)
- net OE_N: now reaches IC1.U17 (IO_L19P_T3_A10_D26_14)
- net OE_N: now also IC2.13 (OE_N)
- net SIWU_N: now reaches IC1.V14 (IO_L23P_T3_A03_D19_14)
- net SIWU_N: now also IC2.10 (SIWU_N)
- net RXF_N: now reaches IC1.V16 (IO_L21P_T3_DQS_14)
- net RXF_N: now also IC2.9 (RXF_N)
- net p31_FPGA: now reaches IC1.W14 (IO_L23N_T3_A02_D18_14)
- net p31_FPGA: now also R5.2, R7.2
- net p30: now reaches IC1.W15 (IO_L24P_T3_A01_D17_14)
- net p30: now also IC2.75 (DATA_30)
- net p29: now reaches IC1.W16 (IO_L24N_T3_A00_D16_14)
- net p29: now also IC2.74 (DATA_29)
- net p28: now reaches IC1.W17 (IO_L20P_T3_A08_D24_14)
- net p28: now also IC2.73 (DATA_28)
- net p27: now reaches IC1.W18 (IO_L20N_T3_A07_D23_14)
- net p27: now also IC2.72 (DATA_27)
- new net: C193.2, IC2.31 (TODN)
- new net: C153.2, IC2.2 (AVDD), IC2.3 (VD10_1), IC2.30 (VD10_2), IC2.33 (VD10_3), IC2.39 (DV10), IC2.48 (VD10_4)
- new net: IC2.37 (VBUS), R16.1, R17.2
- new net: C197.2, IC2.32 (TODP)
- new net: IC2.16 (WAKEUP_N), TP58.1
- new net: C198.2, IC2.15 (RESET_N), R18.2, TP67.1
- new net: IC2.17 (GPIO0), TP61.1
- new net: IC2.18 (GPIO1), TP62.1
- new net: IC2.27 (RREF), R15.2
- new net: J1.B5 (CC2), R73.1
- new net: R5.1, R6.2
- new net: J1.A5 (CC1), R70.2
- new net DN: IC2.25 (DM), J1.A7 (DN1), J1.B7 (DN2)
- new net DP: IC2.23 (DP), J1.A6 (DP1), J1.B6 (DP2)
- new net FTDI_XI: C199.2, IC2.21 (XI), Y2.3 (CRYSTAL_2)
- new net FTDI_XO: C200.1, IC2.22 (XO), Y2.1 (CRYSTAL_1)
- new net SSRXN: IC2.34 (RIDN), J1.A10 (SSRXN2)
- new net SSRXP: IC2.35 (RIDP), J1.A11 (SSRXP2)
- new net SSTXN: C193.1, J1.A3 (SSTXN1)
- new net SSTXP: C197.1, J1.A2 (SSTXP1)
- new net p31: IC2.76 (DATA_31), R7.1
- no-connect marks 109 -> 105
Other:
- note added: "USB"
- note removed: "FPGA IO and USB"
- moved on the sheet: C163, C164, C172, C173, C84, C86, IC1A, IC1B, IC1C
